File: PCB/YAPC_HEATER_TEMP.sch (KiCad schematic (older format))
At the start: 0 parts

Commit message: Create sheet hierarchy
Add more sheets into the project, ready for the various components to be
added
Other:
- note removed: "CPU Block: STM32F407IEH6\nStepper Driver: A4988SETTR-T (5x)\nLAN PHY: LAN8720A\nLAN CLK: 501AAA50M0000DAG\nLAN RJ45: ARJC01-111002AR\nMOSFETs:\nPSU (Switching): L7987\nMicro SD Card Holder:"
Changed lines of the file:
@@
 EELAYER 25 0
 EELAYER END
-$Descr A3 16535 11693
+$Descr A4 11693 8268
 encoding utf-8
-Sheet 1 3
-Title "Yet Another Printer Controller"
+Sheet 1 6
+Title ""
 Date ""
 Rev ""
-Comp "Studio CM"
+Comp ""
 Comment1 ""
 Comment2 ""
@@
 Comment4 ""
 $EndDescr
-Text Notes 5050 3600 0    60   ~ 0
-CPU Block: STM32F407IEH6\nStepper Driver: A4988SETTR-T (5x)\nLAN PHY: LAN8720A\nLAN CLK: 501AAA50M0000DAG\nLAN RJ45: ARJC01-111002AR\nMOSFETs:\nPSU (Switching): L7987\nMicro SD Card Holder:
-$Sheet
-S 9400 5900 2250 1650
-U 55B5AEC5
-F0 "YAPC Primary CPU" 60
-F1 "YAPC_PriCPU.sch" 60
-$EndSheet
-$Sheet
-S 12000 5900 2150 1650
-U 55BDA0EC
-F0 "YAPC LAN Interface" 60
-F1 "YAPC_LAN.sch" 60
-$EndSheet
 $EndSCHEMATC
